File: Keyboard_Design.kicad_sch (KiCad schematic)
At the start: 70 parts

Commit message: Updates to base keyboard to include changes to controller for LED's, and key switches
Parts:
- added C? (x2): 22pf, symbol Device:C
- added C?: 100uf, symbol Device:C
- added D? (x70): DIODE, symbol pspice:DIODE
- added DS?: OLED-128O064D, Display:OLED-128O064D, symbol Display_Graphic:OLED-128O064D
- added J?: Micro_SD_Card, symbol Connector:Micro_SD_Card
- added J?: USB3_A, symbol Connector:USB3_A
- added SW? (x62): CherryMX, symbol CherryMX:CherryMX
- added TP? (x7): TestPoint, symbol Connector:TestPoint
- added U?: ESP8266EX, Package_DFN_QFN:QFN-32-1EP_5x5mm_P0.5mm_EP3.45x3.45mm, symbol MCU_Espressif:ESP8266EX
- added U?: FT232RL, Package_SO:SSOP-28_5.3x10.2mm_P0.65mm, symbol Interface_USB:FT232RL
- added U?: ATmega2560-16A, Package_QFP:TQFP-100_14x14mm_P0.5mm, symbol MCU_Microchip_ATmega:ATmega2560-16A
- added U?: RN4871, RF_Module:Microchip_RN4871, symbol RF_Bluetooth:RN4871
- added Y?: Crystal, symbol Device:Crystal
Connections:
- net Earth: now also U?.21 (GND), U?.3 (PE0), U?.5 (GND), C?.1, C?.2, C?.2, TP?.1
- net VDD: now also U?.18 (AVCC), U?.20 (AREF), U?.4 (VCC), U?.6 (PE1), C?.2, TP?.1
- net at D?.4 (DIN), U?.25 (PC2): now also TP?.1
- net at U?.15 (PB3): now also TP?.1
- net at U?.16 (PB4): now also TP?.1
- net at U?.17 (PB5): now also TP?.1
- net at 10K-1%.2, U?.29 (~{RESET}/PC6): now also TP?.1
- net at U?.7 (XTAL1/PB6): now also C?.1, Y?.2
- net at U?.8 (XTAL2/PB7): now also C?.1, Y?.1
- new net: D?.2 (A), SW?.2 (x62)
- new net: DS?.1 (GND), DS?.30 (GND)
- new net: U?.10 (VCC), U?.31 (VCC), U?.61 (VCC), U?.80 (VCC)
- new net: U?.11 (GND), U?.32 (GND), U?.62 (GND), U?.81 (GND), U?.99 (GND)
- new net Col1: D?.1 (K), D?.1 (K), D?.1 (K), D?.1 (K), D?.1 (K), D?.1 (K), D?.1 (K), D?.1 (K), D?.1 (K), D?.1 (K), D?.1 (K), D?.1 (K), D?.1 (K), D?.1 (K)
- new net Col2: D?.1 (K), D?.1 (K), D?.1 (K), D?.1 (K), D?.1 (K), D?.1 (K), D?.1 (K), D?.1 (K), D?.1 (K), D?.1 (K), D?.1 (K), D?.1 (K), D?.1 (K), D?.1 (K)
- new net Col3: D?.1 (K), D?.1 (K), D?.1 (K), D?.1 (K), D?.1 (K), D?.1 (K), D?.1 (K), D?.1 (K), D?.1 (K), D?.1 (K), D?.1 (K), D?.1 (K), D?.1 (K), D?.1 (K)
- new net Col4: D?.1 (K), D?.1 (K), D?.1 (K), D?.1 (K), D?.1 (K), D?.1 (K), D?.1 (K), D?.1 (K), D?.1 (K), D?.1 (K), D?.1 (K), D?.1 (K), D?.1 (K), D?.1 (K)
- new net Col5: D?.1 (K), D?.1 (K), D?.1 (K), D?.1 (K), D?.1 (K), D?.1 (K), D?.1 (K), D?.1 (K), D?.1 (K), D?.1 (K), D?.1 (K), D?.1 (K), D?.1 (K), D?.1 (K)
- new net Row1: SW?.1, SW?.1, SW?.1, SW?.1, SW?.1
- new net Row10: SW?.1, SW?.1, SW?.1, SW?.1
- new net Row11: SW?.1, SW?.1, SW?.1, SW?.1
- new net Row12: SW?.1, SW?.1, SW?.1, SW?.1
- new net Row13: SW?.1, SW?.1, SW?.1
- new net Row14: SW?.1, SW?.1
- new net Row2: SW?.1, SW?.1, SW?.1, SW?.1, SW?.1
- new net Row3: SW?.1, SW?.1, SW?.1, SW?.1, SW?.1
- new net Row4: SW?.1, SW?.1, SW?.1, SW?.1, SW?.1
- new net Row5: SW?.1, SW?.1, SW?.1, SW?.1, SW?.1
- new net Row6: SW?.1, SW?.1, SW?.1, SW?.1, SW?.1
- new net Row7: SW?.1, SW?.1, SW?.1, SW?.1, SW?.1
- new net Row8: SW?.1, SW?.1, SW?.1, SW?.1, SW?.1
- new net Row9: SW?.1, SW?.1, SW?.1, SW?.1, SW?.1
Other:
- moved on the sheet: D?
